File: 03-smd-project/tesla_smps.kicad_pcb (KiCad board)
At the start: 2 copper layers, 110.5 x 90.8 mm, 112 parts, among them J1 OUTPUT: 25.8 VDC/20 W, P1 Line1, P2 Line2, T1 2SK1317, T2 2N2222, T3 2N2222, U1 LTV-817, U2 LTV-817

Commit message: Working on documentation
Other:
- board text added: "https://github.com/devfabiosilva/TeslaSMPS"
- board text removed: "https://github.com/devfabiosilva/myTeslaSMPS"
Changed lines of the file:
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@@
     (pad_to_mask_clearance 0.2)
     (pcbplotparams
-      (layerselection 0x00014b0_ffffffff)
+      (layerselection 0x00010f0_ffffffff)
       (disableapertmacros false)
       (usegerberextensions false)
@@
       (drillshape 0)
       (scaleselection 1)
-      (outputdirectory "gerber/")
+      (outputdirectory "../02-schematic_and_gerber_files/gerber/")
     )
   )
@@
     (effects (font (size 0.8 0.8) (thickness 0.15)))
   )
-  (gr_text "https://github.com/devfabiosilva/myTeslaSMPS" (at 156.21 144.78) (layer "F.SilkS")
+  (gr_text "https://github.com/devfabiosilva/TeslaSMPS" (at 156.21 144.78) (layer "F.SilkS")
     (effects (font (size 1 1) (thickness 0.15)))
   )
@@
   )
   (dimension (type aligned) (layer "Eco2.User")
-    (pts (xy 76.835 147.32) (xy 192.405 147.32))
-    (height 5.08)
-    (gr_text "115.5700 mm" (at 134.62 151.25) (layer "Eco2.User")
+    (pts (xy 195.58 59.69) (xy 195.58 149.86))
+    (height -1.27)
+    (gr_text "90.1700 mm" (at 195.7 104.775 90) (layer "Eco2.User")
       (effects (font (size 1 1) (thickness 0.15)))
     )
-    (format (units 2) (units_format 1) (precision 4))
-    (style (thickness 0.15) (arrow_length 1.27) (text_position_mode 0) (extension_height 0.58642) (extension_offset 0) keep_text_aligned)
+    (format (units 3) (units_format 1) (precision 4))
+    (style (thickness 0.1) (arrow_length 1.27) (text_position_mode 0) (extension_height 0.58642) (extension_offset 0.5) keep_text_aligned)
   )
   (dimension (type aligned) (layer "Eco2.User")
-    (pts (xy 194.945 60.96) (xy 194.31 145.415))
-    (height -5.079855)
-    (gr_text "84.4574 mm" (at 198.557244 103.217047 89.56921278) (layer "Eco2.User")
+    (pts (xy 77.47 154.94) (xy 187.96 154.94))
+    (height 0)
+    (gr_text "110.4900 mm" (at 132.715 153.79) (layer "Eco2.User")
       (effects (font (size 1 1) (thickness 0.15)))
     )
-    (format (units 2) (units_format 1) (precision 4))
-    (style (thickness 0.15) (arrow_length 1.27) (text_position_mode 0) (extension_height 0.58642) (extension_offset 0) keep_text_aligned)
+    (format (units 3) (units_format 1) (precision 4))
+    (style (thickness 0.1) (arrow_length 1.27) (text_position_mode 0) (extension_height 0.58642) (extension_offset 0.5) keep_text_aligned)
   )
   (segment (start 168.785 62.99) (end 170.18 62.99) (width 0.5) (layer "F.Cu") (net 1))
